Commit message: format xacro

File: xacro/test.xacro (robot description, xacro)
@@ -3,29 +3,29 @@
   <link name="base_footprint"/>
   <link name="base_link">
-      <visual>
-        <origin rpy="0 0 0 " xyz="0 0 0.005"/>
-        <geometry>
-            <box size="0.4 0.4 0.01"/>
-        </geometry>
-      </visual>
-      <collision>
-        <origin rpy="0 0 0 " xyz="0 0 0.005"/>
-        <geometry>
-          <box size="0.4 0.4 0.01"/>
-        </geometry>
-      </collision>
-      <inertial>
-        <origin rpy="0 0 0 " xyz="0 0 0.005"/>
-        <geometry>
-          <box size="0.4 0.4 0.01"/>
-        </geometry>
-        <mass value="100"/>
-        <inertia ixx="1.0265" ixy="0" ixz="0" iyy="1.3944999999999999" iyz="0" izz="2.1320000000000001"/>
-      </inertial>
+    <visual>
+      <origin rpy="0 0 0 " xyz="0 0 0.005"/>
+      <geometry>
+        <box size="0.4 0.4 0.01"/>
+      </geometry>
+    </visual>
+    <collision>
+      <origin rpy="0 0 0 " xyz="0 0 0.005"/>
+      <geometry>
+        <box size="0.4 0.4 0.01"/>
+      </geometry>
+    </collision>
+    <inertial>
+      <origin rpy="0 0 0 " xyz="0 0 0.005"/>
+      <geometry>
+        <box size="0.4 0.4 0.01"/>
+      </geometry>
+      <mass value="100"/>
+      <inertia ixx="1.0265" ixy="0" ixz="0" iyy="1.3944999999999999" iyz="0" izz="2.1320000000000001"/>
+    </inertial>
   </link>
   <joint name="base_joint" type="fixed">
-      <parent link="base_footprint"/>
-      <child link="base_link"/>
-      <origin rpy="0 0 0" xyz="0 0 0"/>
+    <parent link="base_footprint"/>
+    <child link="base_link"/>
+    <origin rpy="0 0 0" xyz="0 0 0"/>
   </joint>
   <xacro:macro name="wheel" params="name">
@@ -34,38 +34,38 @@
         <origin rpy="0 0 0" xyz="0 0 0"/>
         <geometry>
-            <cylinder length="0.05" radius="0.11"/>
+          <cylinder length="0.05" radius="0.11"/>
         </geometry>
       </visual>
       <collision>
-          <origin rpy="0 0 0" xyz="0 0 0"/>
-          <geometry>
-              <cylinder length="0.05" radius="0.11"/>
-          </geometry>
+        <origin rpy="0 0 0" xyz="0 0 0"/>
+        <geometry>
+          <cylinder length="0.05" radius="0.11"/>
+        </geometry>
       </collision>
       <inertial>
         <origin rpy="0 0 0" xyz="0 0 0"/>
         <geometry>
-            <cylinder length="0.05" radius="0.11"/>
+          <cylinder length="0.05" radius="0.11"/>
         </geometry>
-          <mass value="3.5"/>
-          <inertia ixx="0.0267" ixy="0" ixz="0" iyy="0.0267" iyz="0" izz="0.0506"/>
+        <mass value="3.5"/>
+        <inertia ixx="0.0267" ixy="0" ixz="0" iyy="0.0267" iyz="0" izz="0.0506"/>
       </inertial>
     </link>
   </xacro:macro>
   <xacro:wheel name="one"/>
-  <!-- <xacro:wheel name="two"/>
+<!--   <xacro:wheel name="two"/>
   <xacro:include filename="$(find gazebo_ros_motors)/xacro/joint_motor.xacro"/>
-  <xacro:joint_motor motor_name="one_motor" parent_link="base_link" child_link="one_wheel_link">
+  <xacro:joint_motor child_link="one_wheel_link" motor_name="one_motor" parent_link="base_link">
     <xacro:property name="params_yaml" value="$(find gazebo_ros_motors)/params/joint_motor.yaml"/>
-    <origin xyz="0 0 0.2" rpy="0 0 0"/>
+    <origin rpy="0 0 0" xyz="0 0 0.2"/>
   </xacro:joint_motor>
-  <xacro:joint_motor motor_name="two_motor" parent_link="base_link" child_link="two_wheel_link">
+  <xacro:joint_motor child_link="two_wheel_link" motor_name="two_motor" parent_link="base_link">
     <xacro:property name="params_yaml" value="$(find gazebo_ros_motors)/params/joint_motor.yaml"/>
-    <origin xyz="0 0 0.4" rpy="0 0 0"/>
+    <origin rpy="0 0 0" xyz="0 0 0.4"/>
   </xacro:joint_motor> -->
   <xacro:include filename="$(find gazebo_ros_motors)/xacro/dc_motor.xacro"/>
-  <xacro:dc_motor motor_name="dc_motor" parent_link="base_link" child_link="one_wheel_link">
+  <xacro:dc_motor child_link="one_wheel_link" motor_name="dc_motor" parent_link="base_link">
     <xacro:property name="params_yaml" value="$(find gazebo_ros_motors)/params/dc_motor.yaml"/>
-    <origin xyz="0 0 0.2" rpy="0 0 0"/>
+    <origin rpy="0 0 0" xyz="0 0 0.2"/>
   </xacro:dc_motor>
 </robot>
